File: kicad/Retro_Bubble_LED_Watch/_autosave-Retro_Bubble_LED_Watch.kicad_sch (KiCad schematic)
At the start: 21 parts, among them J2 AVR ISP Connector, SW1 MODE, SW2 UP, U2 ATmega328PB-A, U3 DS1337S+

Commit message: new layout
Parts:
- removed J2: AVR ISP Connector, Connector_PinHeader_2.54mm:PinHeader_2x03_P2.54mm_Vertical_SMD, symbol Connector_Generic:Conn_02x03_Odd_Even
Changed lines of the file:
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@@
-    )
-  )
-  (symbol (lib_id "Connector_Generic:Conn_02x03_Odd_Even") (at 254 85.09 0) (unit 1)
-    (in_bom yes) (on_board yes) (dnp no) (fields_autoplaced)
-    (property "Reference" "J2" (at 255.27 76.2 0)
-      (effects (font (size 1.27 1.27)))
-    )
-    (property "Value" "AVR ISP Connector" (at 255.27 78.74 0)
-      (effects (font (size 1.27 1.27)))
-    )
-    (property "Footprint" "Connector_PinHeader_2.54mm:PinHeader_2x03_P2.54mm_Vertical_SMD" (at 254 85.09 0)
-      (effects (font (size 1.27 1.27)) hide)
-    )
-    (property "Datasheet" "~" (at 254 85.09 0)
-      (effects (font (size 1.27 1.27)) hide)
-    )
-    (pin "2")
-    (pin "3")
-    (pin "4")
-    (pin "1")
-    (pin "5")
-    (pin "6")
-    (instances
-      (project "Retro_Bubble_LED_Watch"
-        (path "/241adb6f-f268-45e9-b7ae-ba5c9ee53a74"
-          (reference "J2") (unit 1)
-        )
-      )
     )
   )
